File: hardware/timetwister.brd (EAGLE design)
At the start: 19.6 x 100.1 mm, 41 parts, among them IC1 PIC16F1825SO14, IC3 LM358D

Commit message: asd
Parts:
- moved LED1 18.2 mm to (17.8, 27.9)
- moved LED5 14.2 mm to (20.6, 14.0)
- moved LED4 4.83 mm to (15.7, 14.0)
- moved LED2 4.83 mm to (6.10, 14.0)
- moved LED3 4.83 mm to (10.9, 14.0)
- flipped POWER to the bottom
- renumbered JP1 to POWER
Connections:
- net LED1: now also LED2.A, LED5.K; no longer LED1.A, LED4.K
- net LED2: now also LED3.K, LED4.A; no longer LED2.K, LED3.A
- net N$12: now also LED1.A; no longer LED5.A
- net N$14: now also LED2.K, LED3.A, LED4.K, LED5.A; no longer LED1.K, LED2.A, LED3.K, LED4.A
- net N$9: now also LED1.K; no longer LED5.K
