File: hardware/timetwister.sch (EAGLE design)
At the start: 41 parts, among them IC1 PIC16F1825SO14, IC3 LM358D

Commit message: asd
Parts:
- renumbered JP1 to POWER
Connections:
- net LED1: now also LED2.A, LED5.C; no longer LED1.A, LED4.C
- net LED2: now also LED3.C, LED4.A; no longer LED2.C, LED3.A
- net N$12: now also LED1.A; no longer LED5.A
- net N$14: now also LED2.C, LED3.A, LED4.C, LED5.A; no longer LED1.C, LED2.A, LED3.C, LED4.A
- net N$9: now also LED1.C; no longer LED5.C
Other:
- moved on the sheet: LED1, LED2, LED3, LED4, LED5
Changed lines of the file:
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@@
 <part name="GND11" library="supply1" deviceset="GND" device=""/>
 <part name="GND12" library="supply1" deviceset="GND" device=""/>
-<part name="LED1" library="led" deviceset="LED" device="3MM"/>
 <part name="LED2" library="led" deviceset="LED" device="3MM"/>
 <part name="LED3" library="led" deviceset="LED" device="3MM"/>
 <part name="LED4" library="led" deviceset="LED" device="3MM"/>
+<part name="LED5" library="led" deviceset="LED" device="3MM"/>
 <part name="R1" library="rcl" deviceset="R-EU_" device="R0805"/>
-<part name="JP1" library="pinhead" deviceset="PINHD-2X5" device=""/>
+<part name="POWER" library="pinhead" deviceset="PINHD-2X5" device=""/>
 <part name="SUPPLY2" library="supply2" deviceset="+12V" device=""/>
 <part name="GND13" library="supply1" deviceset="GND" device=""/>
@@
 <part name="GND6" library="supply1" deviceset="GND" device=""/>
 <part name="GND7" library="supply1" deviceset="GND" device=""/>
-<part name="LED5" library="led" deviceset="LED" device="3MM"/>
+<part name="LED1" library="led" deviceset="LED" device="3MM"/>
 <part name="R2" library="rcl" deviceset="R-EU_" device="R0805"/>
 <part name="GND8" library="supply1" deviceset="GND" device=""/>
@@
 <instance part="GND11" gate="1" x="-27.94" y="-2.54"/>
 <instance part="GND12" gate="1" x="-27.94" y="-50.8"/>
-<instance part="LED1" gate="G$1" x="297.18" y="101.6"/>
-<instance part="LED2" gate="G$1" x="297.18" y="88.9"/>
-<instance part="LED3" gate="G$1" x="304.8" y="86.36" rot="R180"/>
-<instance part="LED4" gate="G$1" x="304.8" y="99.06" rot="R180"/>
+<instance part="LED2" gate="G$1" x="297.18" y="101.6"/>
+<instance part="LED3" gate="G$1" x="297.18" y="88.9"/>
+<instance part="LED4" gate="G$1" x="304.8" y="86.36" rot="R180"/>
+<instance part="LED5" gate="G$1" x="304.8" y="99.06" rot="R180"/>
 <instance part="R1" gate="G$1" x="287.02" y="93.98" rot="R180"/>
-<instance part="JP1" gate="A" x="-22.86" y="177.8"/>
+<instance part="POWER" gate="A" x="-22.86" y="177.8"/>
 <instance part="SUPPLY2" gate="+12V" x="25.4" y="198.12"/>
 <instance part="GND13" gate="1" x="-33.02" y="157.48"/>
@@
 <instance part="IC3" gate="B" x="88.9" y="-7.62"/>
 <instance part="GND7" gate="1" x="71.12" y="-15.24"/>
-<instance part="LED5" gate="G$1" x="106.68" y="71.12"/>
+<instance part="LED1" gate="G$1" x="106.68" y="71.12"/>
 <instance part="R2" gate="G$1" x="106.68" y="58.42" rot="R270"/>
 <instance part="GND8" gate="1" x="106.68" y="48.26"/>
@@
 </segment>
 <segment>
-<pinref part="JP1" gate="A" pin="3"/>
+<pinref part="POWER" gate="A" pin="3"/>
 <wire x1="-25.4" y1="180.34" x2="-33.02" y2="180.34" width="0.1524" layer="91"/>
 <wire x1="-33.02" y1="180.34" x2="-33.02" y2="177.8" width="0.1524" layer="91"/>
-<pinref part="JP1" gate="A" pin="7"/>
+<pinref part="POWER" gate="A" pin="7"/>
 <wire x1="-33.02" y1="177.8" x2="-33.02" y2="175.26" width="0.1524" layer="91"/>
 <wire x1="-33.02" y1="175.26" x2="-25.4" y2="175.26" width="0.1524" layer="91"/>
-<pinref part="JP1" gate="A" pin="5"/>
+<pinref part="POWER" gate="A" pin="5"/>
 <wire x1="-25.4" y1="177.8" x2="-33.02" y2="177.8" width="0.1524" layer="91"/>
 <junction x="-33.02" y="177.8"/>
 <wire x1="-33.02" y1="175.26" x2="-33.02" y2="165.1" width="0.1524" layer="91"/>
 <junction x="-33.02" y="175.26"/>
-<pinref part="JP1" gate="A" pin="4"/>
+<pinref part="POWER" gate="A" pin="4"/>
 <wire x1="-17.78" y1="180.34" x2="-10.16" y2="180.34" width="0.1524" layer="91"/>
 <wire x1="-10.16" y1="180.34" x2="-10.16" y2="177.8" width="0.1524" layer="91"/>
-<pinref part="JP1" gate="A" pin="8"/>
+<pinref part="POWER" gate="A" pin="8"/>
 <wire x1="-10.16" y1="177.8" x2="-10.16" y2="175.26" width="0.1524" layer="91"/>
 <wire x1="-10.16" y1="175.26" x2="-17.78" y2="175.26" width="0.1524" layer="91"/>
-<pinref part="JP1" gate="A" pin="6"/>
+<pinref part="POWER" gate="A" pin="6"/>
 <wire x1="-17.78" y1="177.8" x2="-10.16" y2="177.8" width="0.1524" layer="91"/>
 <junction x="-10.16" y="177.8"/>
@@
 <net name="LED1" class="0">
 <segment>
-<pinref part="LED1" gate="G$1" pin="A"/>
+<pinref part="LED2" gate="G$1" pin="A"/>
 <wire x1="297.18" y1="109.22" x2="297.18" y2="104.14" width="0.1524" layer="91"/>
-<pinref part="LED4" gate="G$1" pin="C"/>
+<pinref part="LED5" gate="G$1" pin="C"/>
 <wire x1="304.8" y1="104.14" x2="304.8" y2="109.22" width="0.1524" layer="91"/>
 <wire x1="304.8" y1="109.22" x2="297.18" y2="109.22" width="0.1524" layer="91"/>
@@
 <segment>
 <pinref part="R1" gate="G$1" pin="1"/>
-<pinref part="LED1" gate="G$1" pin="C"/>
+<pinref part="LED2" gate="G$1" pin="C"/>
 <wire x1="292.1" y1="93.98" x2="297.18" y2="93.98" width="0.1524" layer="91"/>
 <wire x1="297.18" y1="93.98" x2="297.18" y2="96.52" width="0.1524" layer="91"/>
-<pinref part="LED4" gate="G$1" pin="A"/>
+<pinref part="LED5" gate="G$1" pin="A"/>
 <wire x1="297.18" y1="93.98" x2="304.8" y2="93.98" width="0.1524" layer="91"/>
 <wire x1="304.8" y1="93.98" x2="304.8" y2="96.52" width="0.1524" layer="91"/>
 <junction x="297.18" y="93.98"/>
-<pinref part="LED2" gate="G$1" pin="A"/>
+<pinref part="LED3" gate="G$1" pin="A"/>
 <wire x1="297.18" y1="93.98" x2="297.18" y2="91.44" width="0.1524" layer="91"/>
-<pinref part="LED3" gate="G$1" pin="C"/>
+<pinref part="LED4" gate="G$1" pin="C"/>
 <wire x1="304.8" y1="93.98" x2="304.8" y2="91.44" width="0.1524" layer="91"/>
 <junction x="304.8" y="93.98"/>
@@
 <net name="LED2" class="0">
 <segment>
-<pinref part="LED2" gate="G$1" pin="C"/>
+<pinref part="LED3" gate="G$1" pin="C"/>
 <wire x1="297.18" y1="83.82" x2="297.18" y2="81.28" width="0.1524" layer="91"/>
-<pinref part="LED3" gate="G$1" pin="A"/>
+<pinref part="LED4" gate="G$1" pin="A"/>
 <wire x1="297.18" y1="81.28" x2="304.8" y2="81.28" width="0.1524" layer="91"/>
 <wire x1="304.8" y1="81.28" x2="304.8" y2="83.82" width="0.1524" layer="91"/>
@@
 <net name="N$13" class="0">
 <segment>
-<pinref part="JP1" gate="A" pin="1"/>
+<pinref part="POWER" gate="A" pin="1"/>
 <wire x1="-25.4" y1="182.88" x2="-33.02" y2="182.88" width="0.1524" layer="91"/>
 <wire x1="-33.02" y1="182.88" x2="-33.02" y2="190.5" width="0.1524" layer="91"/>
 <wire x1="-33.02" y1="190.5" x2="-10.16" y2="190.5" width="0.1524" layer="91"/>
 <wire x1="-10.16" y1="190.5" x2="-10.16" y2="182.88" width="0.1524" layer="91"/>
-<pinref part="JP1" gate="A" pin="2"/>
+<pinref part="POWER" gate="A" pin="2"/>
 <wire x1="-10.16" y1="182.88" x2="-17.78" y2="182.88" width="0.1524" layer="91"/>
 <pinref part="D1" gate="G$1" pin="A"/>
@@
 <segment>
 <pinref part="R2" gate="G$1" pin="1"/>
-<pinref part="LED5" gate="G$1" pin="C"/>
+<pinref part="LED1" gate="G$1" pin="C"/>
 <wire x1="106.68" y1="63.5" x2="106.68" y2="66.04" width="0.1524" layer="91"/>
 </segment>
@@
 <segment>
 <pinref part="IC1" gate="G$1" pin="RC3/SS#"/>
-<pinref part="LED5" gate="G$1" pin="A"/>
+<pinref part="LED1" gate="G$1" pin="A"/>
 <wire x1="121.92" y1="91.44" x2="106.68" y2="91.44" width="0.1524" layer="91"/>
 <wire x1="106.68" y1="91.44" x2="106.68" y2="73.66" width="0.1524" layer="91"/>

Commit message: sdfdsfa
Connections:
- removed net N$12: IC1.RC3/SS#, LED1.A
- new net LED0: IC1.RA1/ICPCLK, ICSP.ICSP_CLK/PGC, LED1.A
- net LED1: now also IC1.RA5; no longer IC1.RA0/ICSPDAT, ICSP.ICSP_DAT/PGD
- net LED2: now also IC1.RC3/SS#; no longer IC1.RA1/ICPCLK, ICSP.ICSP_CLK/PGC
- net LED_COM: now also IC1.RA0/ICSPDAT, ICSP.ICSP_DAT/PGD; no longer IC1.RA5
Changed lines of the file:
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@@
 </segment>
 <segment>
-<pinref part="IC1" gate="G$1" pin="RA0/ICSPDAT"/>
-<pinref part="ICSP" gate="G$1" pin="ICSP_DAT/PGD"/>
-<wire x1="165.1" y1="104.14" x2="177.8" y2="104.14" width="0.1524" layer="91"/>
-<wire x1="177.8" y1="104.14" x2="187.96" y2="104.14" width="0.1524" layer="91"/>
-<wire x1="177.8" y1="104.14" x2="177.8" y2="116.84" width="0.1524" layer="91"/>
-<junction x="177.8" y="104.14"/>
-<label x="177.8" y="116.84" size="1.778" layer="95" rot="R90"/>
+<pinref part="IC1" gate="G$1" pin="RA5"/>
+<wire x1="121.92" y1="104.14" x2="109.22" y2="104.14" width="0.1524" layer="91"/>
+<label x="106.68" y="104.14" size="1.778" layer="95"/>
 </segment>
 </net>
@@
 </segment>
 <segment>
-<pinref part="IC1" gate="G$1" pin="RA5"/>
-<wire x1="121.92" y1="104.14" x2="109.22" y2="104.14" width="0.1524" layer="91"/>
-<label x="106.68" y="104.14" size="1.778" layer="95"/>
+<pinref part="IC1" gate="G$1" pin="RA0/ICSPDAT"/>
+<pinref part="ICSP" gate="G$1" pin="ICSP_DAT/PGD"/>
+<wire x1="165.1" y1="104.14" x2="177.8" y2="104.14" width="0.1524" layer="91"/>
+<wire x1="177.8" y1="104.14" x2="187.96" y2="104.14" width="0.1524" layer="91"/>
+<wire x1="177.8" y1="104.14" x2="177.8" y2="116.84" width="0.1524" layer="91"/>
+<junction x="177.8" y="104.14"/>
+<label x="177.8" y="116.84" size="1.778" layer="95" rot="R90"/>
 </segment>
 </net>
@@
 </segment>
 <segment>
-<pinref part="ICSP" gate="G$1" pin="ICSP_CLK/PGC"/>
-<pinref part="IC1" gate="G$1" pin="RA1/ICPCLK"/>
-<wire x1="187.96" y1="101.6" x2="180.34" y2="101.6" width="0.1524" layer="91"/>
-<wire x1="180.34" y1="101.6" x2="165.1" y2="101.6" width="0.1524" layer="91"/>
-<wire x1="180.34" y1="101.6" x2="180.34" y2="116.84" width="0.1524" layer="91"/>
-<junction x="180.34" y="101.6"/>
-<label x="182.88" y="116.84" size="1.778" layer="95" rot="R90"/>
+<pinref part="IC1" gate="G$1" pin="RC3/SS#"/>
+<wire x1="121.92" y1="91.44" x2="106.68" y2="91.44" width="0.1524" layer="91"/>
+<label x="106.68" y="91.44" size="1.778" layer="95"/>
 </segment>
 </net>
@@
 </segment>
 </net>
-<net name="N$12" class="0">
+<net name="LED0" class="0">
 <segment>
-<pinref part="IC1" gate="G$1" pin="RC3/SS#"/>
 <pinref part="LED1" gate="G$1" pin="A"/>
-<wire x1="121.92" y1="91.44" x2="106.68" y2="91.44" width="0.1524" layer="91"/>
-<wire x1="106.68" y1="91.44" x2="106.68" y2="73.66" width="0.1524" layer="91"/>
+<wire x1="106.68" y1="81.28" x2="106.68" y2="73.66" width="0.1524" layer="91"/>
+<label x="104.14" y="81.28" size="1.778" layer="95"/>
+</segment>
+<segment>
+<pinref part="ICSP" gate="G$1" pin="ICSP_CLK/PGC"/>
+<pinref part="IC1" gate="G$1" pin="RA1/ICPCLK"/>
+<wire x1="187.96" y1="101.6" x2="180.34" y2="101.6" width="0.1524" layer="91"/>
+<wire x1="180.34" y1="101.6" x2="165.1" y2="101.6" width="0.1524" layer="91"/>
+<wire x1="180.34" y1="101.6" x2="180.34" y2="116.84" width="0.1524" layer="91"/>
+<junction x="180.34" y="101.6"/>
+<label x="182.88" y="116.84" size="1.778" layer="95" rot="R90"/>
 </segment>
 </net>

Commit message: sas
Connections:
- new net N$12: POWER.10, POWER.9
Other:
- note added: "CC-NC-BY-SA"
- note added: "DICKY TICKER"
- note added: "Sixty Four Pixels Ltd"
- note added: "Version 1 (15 JAN 2020)"
- moved on the sheet: C2, C3, C4, C5, C6, C7, C8, C9, CLK_IN, CLK_OUT, D1, D2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
