File: hardware/d-ticker.sch (EAGLE design)
At the start: 41 parts, among them IC1 PIC16F1825SO14, IC3 LM358D

Commit message: asasasas
Parts:
- C5: value (none) -> 10n
- R3, R7, R8: value (none) -> 1k
- R4, R9: value (none) -> 4k7
- R5, R6: value (none) -> 10k
- renumbered C7 to R9
Changed lines of the file:
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@@
 <part name="RST_IN" library="thonkiconn" deviceset="WQP-PJ301M-12_JACK" device=""/>
 <part name="D2" library="jasons_stuff" deviceset="0805DIODE" device=""/>
-<part name="R3" library="rcl" deviceset="R-EU_" device="R0805"/>
+<part name="R3" library="rcl" deviceset="R-EU_" device="R0805" value="1k"/>
 <part name="Q1" library="transistor-neu-to92" deviceset="*-NPN-" device="SOT23-BEC" technology="MMBT3904LT1"/>
-<part name="R4" library="rcl" deviceset="R-EU_" device="R0805"/>
+<part name="R4" library="rcl" deviceset="R-EU_" device="R0805" value="4k7"/>
 <part name="P+2" library="supply1" deviceset="VCC" device=""/>
 <part name="Q2" library="transistor-neu-to92" deviceset="*-NPN-" device="SOT23-BEC" technology="MMBT3904LT1"/>
-<part name="R8" library="rcl" deviceset="R-EU_" device="R0805"/>
-<part name="C7" library="rcl" deviceset="R-EU_" device="R0805"/>
+<part name="R8" library="rcl" deviceset="R-EU_" device="R0805" value="1k"/>
+<part name="R9" library="rcl" deviceset="R-EU_" device="R0805" value="4k7"/>
 <part name="P+3" library="supply1" deviceset="VCC" device=""/>
 <part name="D3" library="jasons_stuff" deviceset="0805DIODE" device=""/>
 <part name="IC3" library="linear" deviceset="LM358" device="D"/>
-<part name="R6" library="rcl" deviceset="R-EU_" device="R0805"/>
-<part name="R5" library="rcl" deviceset="R-EU_" device="R0805"/>
-<part name="R7" library="rcl" deviceset="R-EU_" device="R0805"/>
-<part name="C5" library="rcl" deviceset="C-EU" device="C0805"/>
+<part name="R6" library="rcl" deviceset="R-EU_" device="R0805" value="10k"/>
+<part name="R5" library="rcl" deviceset="R-EU_" device="R0805" value="10k"/>
+<part name="R7" library="rcl" deviceset="R-EU_" device="R0805" value="1k"/>
+<part name="C5" library="rcl" deviceset="C-EU" device="C0805" value="10n"/>
 <part name="S1" library="switch-omron" deviceset="10-XX" device=""/>
 <part name="ICSP" library="tag-connect" deviceset="TC2030" device="-MCP-NL"/>
@@
 <instance part="Q2" gate="G$1" x="-10.16" y="-12.7"/>
 <instance part="R8" gate="G$1" x="-22.86" y="-12.7"/>
-<instance part="C7" gate="G$1" x="-7.62" y="-27.94" rot="R90"/>
+<instance part="R9" gate="G$1" x="-7.62" y="-27.94" rot="R90"/>
 <instance part="P+3" gate="VCC" x="-7.62" y="-2.54"/>
 <instance part="D3" gate="G$1" x="-33.02" y="-12.7" rot="R270"/>
@@
 <segment>
 <pinref part="Q2" gate="G$1" pin="E"/>
-<pinref part="C7" gate="G$1" pin="2"/>
+<pinref part="R9" gate="G$1" pin="2"/>
 <wire x1="-7.62" y1="-17.78" x2="-7.62" y2="-20.32" width="0.1524" layer="91"/>
 <wire x1="-7.62" y1="-20.32" x2="-7.62" y2="-22.86" width="0.1524" layer="91"/>
@@
 </segment>
 <segment>
-<pinref part="C7" gate="G$1" pin="1"/>
+<pinref part="R9" gate="G$1" pin="1"/>
 <pinref part="GND12" gate="1" pin="GND"/>
 <wire x1="-7.62" y1="-33.02" x2="-7.62" y2="-38.1" width="0.1524" layer="91"/>

Commit message: dasads
Other:
- note added: "+/- REVERSED"
- note added: "NOT TL072!"
- note added: "SCHMITT TRIGGER INPUT"
Changed lines of the file:
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@@
 <wire x1="213.36" y1="-50.8" x2="213.36" y2="-5.08" width="0.1524" layer="97"/>
 <wire x1="213.36" y1="-5.08" x2="101.6" y2="-5.08" width="0.1524" layer="97"/>
+<text x="86.36" y="15.24" size="6.35" layer="97">NOT TL072!</text>
+<text x="10.16" y="58.42" size="6.35" layer="97">+/- REVERSED</text>
+<text x="-35.56" y="0" size="6.35" layer="97">SCHMITT
+TRIGGER
+INPUT</text>
 </plain>
 <instances>
@@
 </schematic>
 </drawing>
+<compatibility>
+<note version="6.3" minversion="6.2.2" severity="warning">
+Since Version 6.2.2 text objects can contain more than one line,
+which will not be processed correctly with this version.
+</note>
+</compatibility>
 </eagle>

Commit message: dsfsdsf
Other:
- note added: "MOVE CLOCK IN TO RA5 TO ALLOW IOC MOVE LED1 TO RC5"
Changed lines of the file:
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@@
 TRIGGER
 INPUT</text>
+<text x="91.44" y="76.2" size="6.35" layer="97">MOVE CLOCK IN TO RA5 TO ALLOW IOC
+MOVE LED1 TO RC5</text>
 </plain>
 <instances>

Commit message: d
Parts:
- removed D2, D3: 0805DIODE, jasons_stuff:0805DIODE
- removed Q1, Q2: (no value), transistor-neu-to92:MMBT3904LT1-NPN-SOT23-BEC
- removed R3, R8: 1k, rcl:R-EU_R0805
- removed R4, R9: 4k7, rcl:R-EU_R0805
- added C7: (no value), rcl:C-EUC0805
- added D4, D5: (no value), diode:ZENER-DIODESMB
- added D6: 0805DIODE, jasons_stuff:0805DIODE
- added IC9: SN74LVC2G14, jason_eagle6:SN74LVC2G14
- added R10, R11: 4k7, rcl:R-EU_R0805
Connections:
- removed net N$2: D2.P$2, R3.1
- removed net N$3: Q1.B, R3.2
- removed net N$4: D3.P$2, R8.1
- removed net N$5: Q2.B, R8.2
- new net N$16: D4.C, IC9.1A, R10.2
- new net N$17: D5.C, IC9.2A, R11.2
- new net N$20: C7.2, D6.P$2, IC9.VCC
- net CLOCK_IN: now also IC9.1Y; no longer Q1.E, R4.2
- net CLOCK_OUT: now also IC3A.+IN; no longer IC3A.-IN
- net GND: now also C7.1, D4.A, D5.A, IC9.GND; no longer R4.1, R9.1
- net N$1: now also R10.1; no longer D2.P$1
- net N$6: now also IC3A.-IN; no longer IC3A.+IN
- net N$7: now also R11.1; no longer D3.P$1
- net RESET_IN: now also IC9.2Y; no longer Q2.E, R9.2
- net VCC: now also D6.P$1; no longer Q1.C, Q2.C
Other:
- note removed: "+/- REVERSED"
- note removed: "SCHMITT TRIGGER INPUT"
- moved on the sheet: CLK_IN, IC3A, RST_IN

Commit message: various changes per prototype
Parts:
- removed D5: (no value), diode:ZENER-DIODESMB
- removed IC9: SN74LVC2G14, jason_eagle6:SN74LVC2G14
- removed R11: 4k7, rcl:R-EU_R0805
- added D3: (no value), diode:ZENER-DIODESOD80C
- added IC4: LM358D, linear:LM358D
- added R4: 10k, rcl:R-EU_R0805
- C3, C6: device rcl:C-EUC0805 -> rcl:CPOL-EUSMCA
- C5: value 10n -> (none)
- C8: device rcl:CPOL-EUE2-5 -> rcl:C-EUC0805
- C9: value (none) -> 10n; device rcl:CPOL-EUE2-5 -> rcl:C-EUC0805
- D4: device diode:ZENER-DIODESMB -> diode:ZENER-DIODESOD80C
- IC3: value LM358D -> SN74LVC2G14; device linear:LM358D -> jason_eagle6:SN74LVC2G14
- R6: value 10k -> 1k
- R7: value 1k -> 4k7
- renumbered D6 to D2, R10 to R3
Connections:
- removed net N$20: C7.2, D2.P$2, IC9.VCC
- new net N$4: C7.2, D2.P$2, IC3.VCC
- net +12V: now also C3.+, C4.1, C8.1, IC4P.V+; no longer C3.1, C6.1, C8.+, IC3P.V+
- net CLOCK_IN: now also IC3.2Y; no longer IC9.1Y
- net CLOCK_OUT: now also IC4A.+IN; no longer IC3A.+IN
- net GND: now also C3.-, C6.-, C8.2, C9.2, D3.A, IC3.GND, IC4B.+IN, IC4P.V-, R5.1; no longer C3.2, C6.2, C8.-, C9.-, D5.A, IC3B.+IN, IC3P.V-, IC9.GND, R6.1
- net N$10: now also IC4A.OUT, R4.2, R6.1; no longer IC3A.OUT, R5.2, R7.1
- net N$11: now also C9.1, R6.2; no longer C5.1, R7.2
- net N$16: now also D3.C, IC3.2A; no longer D4.C, IC9.1A
- net N$17: now also D4.C, IC3.1A, R7.2; no longer D5.C, IC9.2A, R11.2
- net N$6: now also IC4A.-IN, R4.1, R5.2; no longer IC3A.-IN, R5.1, R6.2
- net N$7: now also R7.1; no longer R11.1
- net N$8: now also IC4B.-IN, IC4B.OUT; no longer IC3B.-IN, IC3B.OUT
- net RESET_IN: now also IC3.1Y; no longer IC9.2Y
- net VCC: now also C5.1, C6.+; no longer C4.1, C9.+
Other:
- note added: "NB MUST BE LM358 NOT TL072!"
- note added: "Version 2 (25 JAN 2025)"
- note removed: "MOVE CLOCK IN TO RA5 TO ALLOW IOC MOVE LED1 TO RC5"
- note removed: "NOT TL072!"
- note removed: "Version 1 (15 JAN 2020)"
- moved on the sheet: C4, C5, D4, R5, R6, R7
