File: hardware/d-ticker.brd (EAGLE design)
At the start: 19.6 x 100.1 mm, 41 parts, among them IC1 PIC16F1825SO14, IC3 LM358D

Commit message: asasasas
Parts:
- C5: value (none) -> 10n
- R3, R7, R8: value (none) -> 1k
- R4, R9: value (none) -> 4k7
- R5, R6: value (none) -> 10k
- renumbered C7 to R9
Changed lines of the file:
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@@
 <attribute name="NAME" x="12.5808" y="25.738" size="1.27" layer="26" font="vector" ratio="20" rot="MR0"/>
 </element>
-<element name="R3" library="rcl" package="R0805" value="" x="11.176" y="21.844" smashed="yes" rot="MR0">
+<element name="R3" library="rcl" package="R0805" value="1k" x="11.176" y="21.844" smashed="yes" rot="MR0">
 <attribute name="NAME" x="12.7" y="19.304" size="1.27" layer="26" font="vector" ratio="20" rot="MR0"/>
 <attribute name="VALUE" x="11.811" y="19.304" size="1.27" layer="28" rot="MR0"/>
@@
 <attribute name="VALUE" x="3.556" y="21.082" size="1.27" layer="28" rot="MR90"/>
 </element>
-<element name="R4" library="rcl" package="R0805" value="" x="5.588" y="27.305" smashed="yes" rot="MR270">
+<element name="R4" library="rcl" package="R0805" value="4k7" x="5.588" y="27.305" smashed="yes" rot="MR270">
 <attribute name="NAME" x="4.318" y="30.861" size="1.27" layer="26" font="vector" ratio="20" rot="MR180"/>
 <attribute name="VALUE" x="8.128" y="27.94" size="1.27" layer="28" rot="MR270"/>
@@
 <attribute name="VALUE" x="3.81" y="5.715" size="1.27" layer="28" rot="MR180"/>
 </element>
-<element name="R8" library="rcl" package="R0805" value="" x="5.715" y="5.715" smashed="yes" rot="MR0">
+<element name="R8" library="rcl" package="R0805" value="1k" x="5.715" y="5.715" smashed="yes" rot="MR0">
 <attribute name="NAME" x="8.89" y="6.985" size="1.27" layer="26" font="vector" ratio="20" rot="MR270"/>
 <attribute name="VALUE" x="6.35" y="3.175" size="1.27" layer="28" rot="MR0"/>
 </element>
-<element name="C7" library="rcl" package="R0805" value="" x="5.715" y="10.795" smashed="yes" rot="MR0">
+<element name="R9" library="rcl" package="R0805" value="4k7" x="5.715" y="10.795" smashed="yes" rot="MR0">
 <attribute name="NAME" x="6.35" y="12.065" size="1.27" layer="26" font="vector" ratio="20" rot="MR0"/>
 <attribute name="VALUE" x="6.35" y="8.255" size="1.27" layer="28" rot="MR0"/>
@@
 <attribute name="NAME" x="11.811" y="13.462" size="1.27" layer="26" font="vector" ratio="20" rot="MR180"/>
 </element>
-<element name="R6" library="rcl" package="R0805" value="" x="18.669" y="6.477" smashed="yes" rot="MR270">
+<element name="R6" library="rcl" package="R0805" value="10k" x="18.669" y="6.477" smashed="yes" rot="MR270">
 <attribute name="NAME" x="19.939" y="10.795" size="1.27" layer="26" font="vector" ratio="20" rot="MR270"/>
 <attribute name="VALUE" x="21.209" y="7.112" size="1.27" layer="28" rot="MR270"/>
 </element>
-<element name="R5" library="rcl" package="R0805" value="" x="21.336" y="6.604" smashed="yes" rot="MR270">
+<element name="R5" library="rcl" package="R0805" value="10k" x="21.336" y="6.604" smashed="yes" rot="MR270">
 <attribute name="NAME" x="22.479" y="10.922" size="1.27" layer="26" font="vector" ratio="20" rot="MR270"/>
 <attribute name="VALUE" x="23.876" y="7.239" size="1.27" layer="28" rot="MR270"/>
 </element>
-<element name="R7" library="rcl" package="R0805" value="" x="21.336" y="2.286" smashed="yes" rot="MR270">
+<element name="R7" library="rcl" package="R0805" value="1k" x="21.336" y="2.286" smashed="yes" rot="MR270">
 <attribute name="NAME" x="17.653" y="3.81" size="1.27" layer="26" font="vector" ratio="20" rot="MR180"/>
 <attribute name="VALUE" x="23.876" y="2.921" size="1.27" layer="28" rot="MR270"/>
 </element>
-<element name="C5" library="rcl" package="C0805" value="" x="13.97" y="1.27" smashed="yes" rot="MR0">
+<element name="C5" library="rcl" package="C0805" value="10n" x="13.97" y="1.27" smashed="yes" rot="MR0">
 <attribute name="NAME" x="9.779" y="1.524" size="1.27" layer="26" font="vector" ratio="20" rot="MR180"/>
 <attribute name="VALUE" x="15.24" y="-1.27" size="1.27" layer="28" rot="MR0"/>
@@
 <signal name="RESET_IN">
 <contactref element="Q2" pad="E"/>
-<contactref element="C7" pad="2"/>
+<contactref element="R9" pad="2"/>
 <contactref element="IC1" pad="3"/>
 <wire x1="6.665" y1="3.64" x2="6.665" y2="1.59" width="0.3048" layer="16"/>
@@
 <contactref element="C5" pad="2"/>
 <contactref element="CLK_OUT" pad="P$3"/>
-<contactref element="C7" pad="1"/>
+<contactref element="R9" pad="1"/>
 <contactref element="R4" pad="1"/>
 <contactref element="CLK_IN" pad="P$3"/>

Commit message: d
Parts:
- removed D2, D3: 0805DIODE, jasons_stuff:0805DIODE
- removed Q1, Q2: (no value), transistor-neu-to92:SOT23-BEC
- removed R3, R8: 1k, rcl:R0805
- removed R4, R9: 4k7, rcl:R0805
- added C7: (no value), rcl:C0805
- added D4, D5: (no value), diode:SMB
- added D6: 0805DIODE, jasons_stuff:0805DIODE
- added IC9: SN74LVC2G14, jason_eagle6:DBV_R-PDSO-G6
- added R10, R11: 4k7, rcl:R0805
Connections:
- removed net N$2: D2.A, R3.1
- removed net N$3: Q1.B, R3.2
- removed net N$4: D3.A, R8.1
- removed net N$5: Q2.B, R8.2
- new net N$16: D4.C, IC9.1, R10.2
- new net N$17: D5.C, IC9.3, R11.2
- new net N$20: C7.2, D6.A, IC9.5
- net CLOCK_IN: now also IC9.6; no longer Q1.E, R4.2
- net CLOCK_OUT: now also IC3.3; no longer IC3.2
- net GND: now also C7.1, D4.A, D5.A, IC9.2; no longer R4.1, R9.1
- net N$1: now also R10.1; no longer D2.C
- net N$6: now also IC3.2; no longer IC3.3
- net N$7: now also R11.1; no longer D3.C
- net RESET_IN: now also IC9.4; no longer Q2.E, R9.2
- net VCC: now also D6.C; no longer Q1.C, Q2.C
Routing:
- net VCC: track 171.7 -> 143.2 mm, vias 3 -> 1
- net N$7: track 7.92 -> 0.00 mm
- net N$3: track 5.28 -> 0.00 mm
- net GND: track 5.09 -> 0.00 mm
- net N$4: track 3.80 -> 0.00 mm
- net CLOCK_IN: track 83.4 -> 79.9 mm
- net N$2: track 2.66 -> 0.00 mm
- net N$1: track 2.65 -> 0.00 mm
- net RESET_IN: track 116.1 -> 113.8 mm
- net CLOCK_OUT: track 104.7 -> 102.6 mm
- net N$5: track 2.07 -> 0.00 mm
- net N$10: track 16.8 -> 14.8 mm
- net N$6: track 10.3 -> 8.56 mm

Commit message: turn mcu
Parts:
- moved C1 12.6 mm to (15.4, 89.2), turned to 180 degrees
- moved C2 1.82 mm to (13.6, 83.3), turned to 0 degrees
- moved IC1 1.27 mm to (13.3, 94.6), turned to 90 degrees
Routing:
- net VCC: track 143.2 -> 127.1 mm
- net LED0: track 83.1 -> 90.7 mm
- net CLOCK_OUT: track 102.6 -> 109.4 mm
- net POT1: track 14.9 -> 21.4 mm
- net POT2: track 31.1 -> 36.0 mm
- net LED1: track 112.8 -> 108.0 mm, vias 5 -> 4
- net RESET_IN: track 113.8 -> 109.4 mm
- net LED2: track 110.4 -> 106.4 mm
- net GND: track 0.00 -> 3.67 mm, vias 9 -> 13
- net LED_COM: track 23.9 -> 27.4 mm
- net N$19: track 90.4 -> 87.8 mm
- net CLOCK_IN: track 79.9 -> 77.9 mm
- net POT3: track 47.2 -> 49.1 mm

Commit message: various changes per prototype
Parts:
- removed D5: (no value), diode:SMB
- removed D6: 0805DIODE, jasons_stuff:0805DIODE
- removed IC9: SN74LVC2G14, jason_eagle6:DBV_R-PDSO-G6
- removed R10, R11: 4k7, rcl:R0805
- added D2: 0805DIODE, jasons_stuff:0805DIODE
- added D3: (no value), diode:SOD80C
- added IC4: LM358D, linear:SO08
- added R3: 4k7, rcl:R0805
- added R4: 10k, rcl:R0805
- C3, C6: device rcl:C0805 -> rcl:SMC_A
- C5: value 10n -> (none)
- C8: device rcl:E2-5 -> rcl:C0805
- C9: value (none) -> 10n; device rcl:E2-5 -> rcl:C0805
- D4: device diode:SMB -> diode:SOD80C
- IC3: value LM358D -> SN74LVC2G14; device linear:SO08 -> jason_eagle6:DBV_R-PDSO-G6
- R6: value 10k -> 1k
- R7: value 1k -> 4k7
- moved C8 69.2 mm to (9.53, 6.35), flipped to the bottom, turned to 270 degrees
- moved C7 64.3 mm to (12.2, 16.4), flipped to the bottom, turned to 90 degrees
- moved C5 52.6 mm to (14.0, 53.8)
- moved C6 46.9 mm to (13.3, 51.6), turned to 0 degrees
- moved C9 43.3 mm to (14.0, 1.40), flipped to the bottom, turned to 0 degrees
- moved D4 38.2 mm to (5.08, 7.62), flipped to the bottom, turned to 90 degrees
- moved R2 20.1 mm to (17.4, 42.9), turned to 0 degrees
- moved LED1 16.7 mm to (20.6, 44.5)
- moved R7 16.3 mm to (5.08, 2.54), turned to 90 degrees
- moved LED2 13.5 mm to (6.10, 27.4)
- moved LED3 13.5 mm to (10.9, 27.4)
- moved LED4 13.5 mm to (15.7, 27.4)
- moved LED5 13.5 mm to (20.6, 27.4)
- moved C4 13.4 mm to (14.1, 65.4), turned to 0 degrees
- moved IC3 13.4 mm to (8.64, 19.1), turned to 90 degrees
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Connections:
- removed net N$20: C7.2, D6.A, IC9.5
- new net N$4: C7.2, D2.A, IC3.5
- net +12V: now also C3.+, C4.1, C8.1, IC4.8; no longer C3.1, C6.1, C8.+, IC3.8
- net CLOCK_IN: now also IC3.4; no longer IC9.6
- net CLOCK_OUT: now also IC4.3; no longer IC3.3
- net GND: now also C3.-, C6.-, C8.2, C9.2, D3.A, IC3.2, IC4.4, IC4.5, R5.1; no longer C3.2, C6.2, C8.-, C9.-, D5.A, IC3.4, IC3.5, IC9.2, R6.1
- net N$1: now also R3.1; no longer R10.1
- net N$10: now also IC4.1, R4.2, R6.1; no longer IC3.1, R5.2, R7.1
- net N$11: now also C9.1, R6.2; no longer C5.1, R7.2
- net N$16: now also D3.C, IC3.3, R3.2; no longer D4.C, IC9.1, R10.2
- net N$17: now also D4.C, IC3.1, R7.2; no longer D5.C, IC9.3, R11.2
- net N$6: now also IC4.2, R4.1, R5.2; no longer IC3.2, R5.1, R6.2
- net N$7: now also R7.1; no longer R11.1
- net N$8: now also IC4.6, IC4.7; no longer IC3.6, IC3.7
- net RESET_IN: now also IC3.6; no longer IC9.4
- net VCC: now also C5.1, C6.+, D2.C; no longer C4.1, C9.+, D6.C
Routing:
- net +12V: track 112.8 -> 78.8 mm, vias 2 -> 4
- net RESET_IN: track 109.4 -> 86.4 mm, vias 3 -> 2
- net LED1: track 108.0 -> 88.7 mm, vias 4 -> 3
- net LED2: track 106.4 -> 88.3 mm, vias 3 -> 2
- net N$17: track 0.00 -> 16.4 mm
- net N$14: track 96.2 -> 80.8 mm
- net VCC: track 127.1 -> 139.0 mm, vias 1 -> 0
- net N$4: track 0.00 -> 8.31 mm
- net CLOCK_IN: track 77.9 -> 86.1 mm
- net LED0: track 90.7 -> 83.2 mm, vias 3 -> 4
- net N$10: track 14.8 -> 21.2 mm, vias 0 -> 2
- net N$1: track 0.00 -> 5.94 mm, vias 0 -> 1
- net N$16: track 0.00 -> 4.74 mm
- net N$7: track 0.00 -> 3.53 mm
- net N$6: track 8.56 -> 11.3 mm
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Other:
- board text added: "2025/hotchk155"
- board text added: "DICKY TICKER V2"
- board text added: "STRIPE -12V"
- board text removed: "+12"
- board text removed: "-12"
- board text removed: "2022/hotchk155"
- board text removed: "DICKY TICKER V1"

Commit message: pcb rev 2
Routing:
- net RESET_IN: track 86.4 -> 86.9 mm
Changed lines of the file:
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@@
 </element>
 <element name="CLK_IN" library="jason_eagle6" package="WQP-PJ301M-ST" value="THONKICONN_STEREO" x="8.509" y="20.32" smashed="yes" rot="R180">
-<attribute name="NAME" x="5.4736" y="12.9968" size="1.27" layer="21" font="vector" ratio="20"/>
+<attribute name="NAME" x="4.5846" y="12.8698" size="1.27" layer="21" font="vector" ratio="20"/>
 </element>
 <element name="CLK_OUT" library="thonkiconn" package="WQP-PJ301M-12_JACK" value="WQP-PJ301M-12_JACK" x="17.78" y="6.35" smashed="yes" rot="R180">
-<attribute name="NAME" x="13.9446" y="10.8458" size="1.27" layer="21" font="vector" ratio="20"/>
+<attribute name="NAME" x="14.7066" y="10.9728" size="1.27" layer="21" font="vector" ratio="20"/>
 </element>
 <element name="RST_IN" library="thonkiconn" package="WQP-PJ301M-12_JACK" value="WQP-PJ301M-12_JACK" x="8.509" y="6.35" smashed="yes" rot="R180">
-<attribute name="NAME" x="5.0546" y="10.8458" size="1.27" layer="21" font="vector" ratio="20"/>
+<attribute name="NAME" x="4.4196" y="11.0998" size="1.27" layer="21" font="vector" ratio="20"/>
 </element>
 <element name="IC4" library="linear" package="SO08" value="LM358D" x="13.843" y="6.731" smashed="yes" rot="MR180">
@@
 <attribute name="MF" value="" x="55.88" y="69.85" size="1.778" layer="27" rot="R90" display="off"/>
 <attribute name="OC_FARNELL" value="176432" x="55.88" y="69.85" size="1.778" layer="27" rot="R90" display="off"/>
-<attribute name="NAME" x="18.542" y="23.876" size="1.27" layer="25" font="vector" ratio="20" rot="R180"/>
+<attribute name="NAME" x="19.177" y="23.876" size="1.27" layer="25" font="vector" ratio="20" rot="R180"/>
 <attribute name="VALUE" x="22.86" y="16.002" size="1.27" layer="27" ratio="10" rot="R90"/>
 </element>
@@
 <wire x1="11.049" y1="94.996" x2="10.16" y2="95.885" width="0.3048" layer="1"/>
 <contactref element="IC3" pad="4"/>
-<wire x1="4.953" y1="24.257" x2="7.62" y2="21.59" width="0.3048" layer="1"/>
-<wire x1="7.62" y1="21.59" x2="9.906" y2="21.59" width="0.3048" layer="1"/>
-<via x="9.906" y="21.59" extent="1-16" drill="0.6"/>
-<wire x1="9.906" y1="21.59" x2="9.906" y2="20.03" width="0.3048" layer="16"/>
+<wire x1="4.953" y1="24.257" x2="6.858" y2="22.479" width="0.3048" layer="1"/>
+<wire x1="6.858" y1="22.479" x2="9.906" y2="22.479" width="0.3048" layer="1"/>
+<via x="9.906" y="22.479" extent="1-16" drill="0.6"/>
+<wire x1="9.906" y1="22.479" x2="9.906" y2="20.03" width="0.3048" layer="16"/>
 <wire x1="9.906" y1="20.03" x2="9.936" y2="20" width="0.3048" layer="16"/>
 </signal>
@@
 <wire x1="9.906" y1="16.891" x2="9.906" y2="18.07" width="0.3048" layer="16"/>
 <wire x1="9.906" y1="18.07" x2="9.936" y2="18.1" width="0.3048" layer="16"/>
-<wire x1="9.906" y1="16.891" x2="9.906" y2="20.32" width="0.3048" layer="1"/>
-<wire x1="9.906" y1="20.32" x2="9.271" y2="20.955" width="0.3048" layer="1"/>
-<wire x1="9.271" y1="20.955" x2="7.366" y2="20.955" width="0.3048" layer="1"/>
-<wire x1="7.366" y1="20.955" x2="4.318" y2="24.003" width="0.3048" layer="1"/>
+<wire x1="9.906" y1="16.891" x2="9.906" y2="21.336" width="0.3048" layer="1"/>
+<wire x1="9.906" y1="21.336" x2="9.398" y2="21.844" width="0.3048" layer="1"/>
+<wire x1="9.398" y1="21.844" x2="6.604" y2="21.844" width="0.3048" layer="1"/>
+<wire x1="6.604" y1="21.844" x2="4.318" y2="24.003" width="0.3048" layer="1"/>
 <wire x1="4.318" y1="67.818" x2="4.318" y2="24.003" width="0.3048" layer="1"/>
 </signal>
@@
 <contactref element="C2" pad="2"/>
 <polygon width="0.3048" layer="16">
-<vertex x="-1.27" y="104.14"/>
-<vertex x="-1.27" y="-5.08"/>
-<vertex x="26.67" y="-5.08"/>
-<vertex x="26.67" y="106.68"/>
-<vertex x="-1.27" y="106.68"/>
+<vertex x="3.556" y="100.33"/>
+<vertex x="3.556" y="0"/>
+<vertex x="23.241" y="0"/>
+<vertex x="23.114" y="99.695"/>
 </polygon>
 <contactref element="IC4" pad="5"/>
 <polygon width="0.4064" layer="1">
-<vertex x="1.27" y="101.6"/>
-<vertex x="1.27" y="-5.08"/>
-<vertex x="24.13" y="-5.08"/>
-<vertex x="24.13" y="101.6"/>
+<vertex x="3.556" y="100.457"/>
+<vertex x="3.556" y="0.127"/>
+<vertex x="23.114" y="0"/>
+<vertex x="23.114" y="100.203"/>
 </polygon>
 <contactref element="R2" pad="2"/>
